File: PCB/flipper-thermal-camera.kicad_pcb (KiCad board)
At the start: 2 copper layers, 67 x 25.2 mm, 27 parts, among them IC1 VEML7700-TT, J1 Conn_01x08, J2 Conn_01x10, U1 MLX90640ESF-BAB-000-SP, U2 XC6206PxxxMR, U3 ICM-20948, U4 SHT31-DIS

Commit message: add arrows and stuff
Other:
- board text added: "IMU"
- board text added: "Light Sensor"
- board text added: "Temp & Humidity Sensor"
- board text added: "Thermal Sensor"
